File: ki/YARC/ConstRegsAndClocks.kicad_sch (KiCad schematic)
At the start: 0 parts

Commit message: Expand ucode RAM test to 4 slices. Much work in KiCad.
Parts:
- added U? (x5): 74LS32, symbol 74xx:74LS32
- added U? (x5): 74HC00, symbol 74xx:74HC00
- added U? (x2): 74HC245, symbol 74xx:74HC245
Connections:
- new net: U?.12, U?.8
- new net: U?.11, U?.12 (B6)
- new net: U?.11, U?.19 (CE)
- new net: U?.19 (CE), U?.8
- new net FLAGS: U?.5
- new net GND: U?.1, U?.1 (A->B), U?.1 (A->B), U?.10 (GND), U?.10 (GND), U?.2, U?.4, U?.5, U?.7 (GND), U?.7 (GND)
- new net S2BUS0: U?.2 (A0)
- new net S2BUS1: U?.3 (A1)
- new net S2BUS10: U?.4 (A2)
- new net S2BUS11: U?.5 (A3)
- new net S2BUS12: U?.6 (A4)
- new net S2BUS13: U?.7 (A5)
- new net S2BUS14: U?.8 (A6)
- new net S2BUS15: U?.9 (A7)
- new net S2BUS2: U?.4 (A2)
- new net S2BUS3: U?.5 (A3)
- new net S2BUS4: U?.6 (A4)
- new net S2BUS5: U?.7 (A5)
- new net S2BUS6: U?.8 (A6)
- new net S2BUS7: U?.11 (B7), U?.12 (B6), U?.13 (B5), U?.14 (B4), U?.15 (B3), U?.16 (B2), U?.17 (B1), U?.18 (B0), U?.9 (A7)
- new net S2BUS8: U?.2 (A0)
- new net S2BUS9: U?.3 (A1)
- new net SYSCLK: U?.1, U?.10, U?.13, U?.4
- new net VCC: U?.14 (VCC), U?.14 (VCC), U?.20 (VCC), U?.20 (VCC)
- new net dsclk: U?.6
- new net grclk: U?.3
- new net src2:0: U?.11 (B7), U?.13
- new net src2:1: U?.10, U?.13 (B5), U?.14 (B4), U?.15 (B3), U?.16 (B2), U?.17 (B1), U?.18 (B0), U?.9
- new net ~{const_en}: U?.12
- new net ~{gr_re}: U?.2
- new net ~{sxt_en}: U?.9
