File: ki/YARC/YARC.kicad_sch (KiCad schematic)
At the start: 0 parts

Commit message: Ongoing development of registers and ALU
Other:
- added sheet ALU (ALU.kicad_sch)
- added sheet ConstRegsAndClocks (ConstRegsAndClocks.kicad_sch)
- added sheet North Central (NorthCentral.kicad_sch)

Commit message: Ongoing development of ALU and registers
Other:
- removed sheet ConstRegsAndClocks
- added sheet ConstantRegisters (ConstRegs.kicad_sch)
