File: ki/YARC/YARC.kicad_sch (KiCad schematic)
At the start: 0 parts

Commit message: All the changes related to the mid-December 2022 K register problem
Other:
- added sheet KludgeSpace (KludgeSpace.kicad_sch)
