File: ki/YARC/KludgeSpace.kicad_sch (KiCad schematic)
At the start: 4 parts, among them J8 6-PIN FROM MCR, U100 74LS32, U101 74LS157, U96 74LS32

Commit message: Various corrections and minor improvements
Parts:
- removed unit 4 of U100
- removed unit 3 of U100
- renumbered U96 to U100
Connections:
- net ~{DST_EN} to U93B renamed ~{DST_EN} to U96B
Other:
- note added: "Temporarily, K8 (dst_wr_en) is directly connected to U101 pin 10. This allows the microcodeto enable register writes when YARC has control."
- note added: "U100C and U100D are in the memory schematic near the bottom - Row D, Column 3."
- note removed: "Temporarily, K(1) bit 0 (dst_wr_en) is directly connected to U101 pin 10. This allows the microcodeto enable register writes when YARC has control."
- note removed: "These gates are part of the memory transceiver control. They are shown on the memory page in row D, column 3."
Changed lines of the file:
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@@
-    (stroke (width 0) (type default) (color 0 0 0 0))
-  )
-  (polyline (pts (xy 86.36 175.26) (xy 27.94 175.26))
     (stroke (width 0) (type default) (color 0 0 0 0))
   )
@@
     (stroke (width 0) (type default) (color 0 0 0 0))
   )
-  (polyline (pts (xy 27.94 175.26) (xy 27.94 190.5))
-    (stroke (width 0) (type default) (color 0 0 0 0))
-  )
   (wire (pts (xy 91.44 86.36) (xy 111.76 86.36))
     (stroke (width 0) (type default) (color 0 0 0 0))
@@
     (stroke (width 0) (type default) (color 0 0 0 0))
   )
-  (polyline (pts (xy 86.36 190.5) (xy 86.36 175.26))
-    (stroke (width 0) (type default) (color 0 0 0 0))
-  )
   (wire (pts (xy 63.5 111.76) (xy 63.5 119.38))
     (stroke (width 0) (type default) (color 0 0 0 0))
@@
     (stroke (width 0) (type default) (color 0 0 0 0))
   )
-  (polyline (pts (xy 27.94 190.5) (xy 86.36 190.5))
-    (stroke (width 0) (type default) (color 0 0 0 0))
-  )
   (wire (pts (xy 78.74 40.64) (xy 55.88 40.64))
     (stroke (width 0) (type default) (color 0 0 0 0))
@@
     (effects (font (size 1.27 1.27)) (justify left bottom))
   )
-  (text "Temporarily, K(1) bit 0 (dst_wr_en)\nis directly connected to U101 pin 10.\nThis allows the microcodeto enable\nregister writes when YARC has control."
+  (text "Temporarily, K8 (dst_wr_en)\nis directly connected to U101 pin 10.\nThis allows the microcodeto enable\nregister writes when YARC has control."
     (at 20.32 129.54 0)
     (effects (font (size 1.27 1.27)) (justify left bottom))
@@
     (effects (font (size 1.27 1.27)) (justify left bottom))
   )
-  (text "These gates are part of the memory transceiver control.\nThey are shown on the memory page in row D, column 3."
-    (at 30.48 195.58 0)
+  (text "U100C and U100D are in the memory schematic\nnear the bottom - Row D, Column 3."
+    (at 88.9 142.24 0)
     (effects (font (size 1.27 1.27)) (justify left bottom))
   )
@@
     )
   )
-  (global_label "~{DST_EN} to U93B" (shape input) (at 127 101.6 0) (fields_autoplaced)
+  (global_label "~{DST_EN} to U96B" (shape input) (at 127 101.6 0) (fields_autoplaced)
     (effects (font (size 1.27 1.27)) (justify left))
     (property "Intersheet References" "${INTERSHEET_REFS}" (id 0) (at 145.1369 101.5206 0)
@@
       (effects (font (size 1.27 1.27)) (justify right) hide)
     )
-  )
-  (symbol (lib_id "74xx:74LS32") (at 73.66 182.88 0) (unit 4)
-    (in_bom yes) (on_board yes)
-    (property "Reference" "U100" (id 0) (at 78.74 177.8 0))
-    (property "Value" "74LS32" (id 1) (at 73.66 182.88 0))
-    (property "Footprint" "" (id 2) (at 73.66 182.88 0)
-      (effects (font (size 1.27 1.27)) hide)
-    )
-    (property "Datasheet" "http://www.ti.com/lit/gpn/sn74LS32" (id 3) (at 73.66 182.88 0)
-      (effects (font (size 1.27 1.27)) hide)
-    )
-    (pin "11")
-    (pin "12")
-    (pin "13")
   )
   (symbol (lib_id "power:VCC") (at 78.74 78.74 0) (unit 1)
@@
     (pin "1")
   )
-  (symbol (lib_id "74xx:74LS32") (at 43.18 182.88 0) (unit 3)
-    (in_bom yes) (on_board yes)
-    (property "Reference" "U100" (id 0) (at 48.26 177.8 0))
-    (property "Value" "74LS32" (id 1) (at 43.18 182.88 0))
-    (property "Footprint" "" (id 2) (at 43.18 182.88 0)
-      (effects (font (size 1.27 1.27)) hide)
-    )
-    (property "Datasheet" "http://www.ti.com/lit/gpn/sn74LS32" (id 3) (at 43.18 182.88 0)
-      (effects (font (size 1.27 1.27)) hide)
-    )
-    (pin "10")
-    (pin "8")
-    (pin "9")
-  )
   (symbol (lib_id "74xx:74LS32") (at 78.74 154.94 0) (unit 1)
     (in_bom yes) (on_board yes)
-    (property "Reference" "U96" (id 0) (at 83.82 149.86 0))
+    (property "Reference" "U100" (id 0) (at 83.82 149.86 0))
     (property "Value" "74LS32" (id 1) (at 78.74 154.94 0))
     (property "Footprint" "" (id 2) (at 78.74 154.94 0)
@@
   (symbol (lib_id "74xx:74LS32") (at 119.38 83.82 0) (mirror x) (unit 2)
     (in_bom yes) (on_board yes)
-    (property "Reference" "U96" (id 0) (at 124.46 78.74 0))
+    (property "Reference" "U100" (id 0) (at 124.46 78.74 0))
     (property "Value" "74LS32" (id 1) (at 119.38 83.82 0))
     (property "Footprint" "" (id 2) (at 119.38 83.82 0)

Commit message: Redesign of ALU control logic
Connections:
- net NANO DECODER 0x02 (bit 1) renamed ACR_CLK NANO DECODER 0x02 (bit 1)
Changed lines of the file:
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@@
     )
   )
-  (global_label "NANO DECODER 0x02 (bit 1)" (shape input) (at 55.88 48.26 180) (fields_autoplaced)
+  (global_label "ACR_CLK NANO DECODER 0x02 (bit 1)" (shape input) (at 55.88 48.26 180) (fields_autoplaced)
     (effects (font (size 1.27 1.27)) (justify right))
-    (property "Intersheet References" "${INTERSHEET_REFS}" (id 0) (at 25.7688 48.1806 0)
+    (property "Intersheet References" "${INTERSHEET_REFS}" (id 0) (at 16.6369 48.1806 0)
       (effects (font (size 1.27 1.27)) (justify right) hide)
     )

Commit message: Yet more cleanup on ALU and flags design
Other:
- note added: "A second 7-pin physical connector is located adjacent to the 6-pin that brings signals from the Nano."
- note added: "Temporarily, K8 (dst_wr_en) is directly connected to U101 pin 10. This allows the microcodeto enable register writes when NANO# has control."
- note removed: "Temporarily, K8 (dst_wr_en) is directly connected to U101 pin 10. This allows the microcodeto enable register writes when YARC has control."
Changed lines of the file:
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@@
   (junction (at 71.12 129.54) (diameter 0) (color 0 0 0 0)
   )
+  (junction (at 73.66 66.04) (diameter 0) (color 0 0 0 0)
+  )
   (wire (pts (xy 104.14 81.28) (xy 111.76 81.28))
     (stroke (width 0) (type default) (color 0 0 0 0))
@@
     (stroke (width 0) (type default) (color 0 0 0 0))
   )
+  (wire (pts (xy 25.4 66.04) (xy 25.4 116.84))
+    (stroke (width 0) (type default) (color 0 0 0 0))
+  )
+  (wire (pts (xy 55.88 53.34) (xy 73.66 53.34))
+    (stroke (width 0) (type default) (color 0 0 0 0))
+  )
+  (wire (pts (xy 60.96 109.22) (xy 60.96 78.74))
+    (stroke (width 0) (type default) (color 0 0 0 0))
+  )
+  (wire (pts (xy 63.5 96.52) (xy 63.5 111.76))
+    (stroke (width 0) (type default) (color 0 0 0 0))
+  )
+  (wire (pts (xy 63.5 129.54) (xy 71.12 129.54))
+    (stroke (width 0) (type default) (color 0 0 0 0))
+  )
+  (wire (pts (xy 71.12 134.62) (xy 71.12 129.54))
+    (stroke (width 0) (type default) (color 0 0 0 0))
+  )
+  (wire (pts (xy 68.58 152.4) (xy 71.12 152.4))
+    (stroke (width 0) (type default) (color 0 0 0 0))
+  )
+  (wire (pts (xy 91.44 86.36) (xy 111.76 86.36))
+    (stroke (width 0) (type default) (color 0 0 0 0))
+  )
+  (wire (pts (xy 58.42 68.58) (xy 58.42 86.36))
+    (stroke (width 0) (type default) (color 0 0 0 0))
+  )
+  (wire (pts (xy 78.74 48.26) (xy 55.88 48.26))
+    (stroke (width 0) (type default) (color 0 0 0 0))
+  )
+  (wire (pts (xy 66.04 111.76) (xy 63.5 111.76))
+    (stroke (width 0) (type default) (color 0 0 0 0))
+  )
+  (wire (pts (xy 78.74 50.8) (xy 55.88 50.8))
+    (stroke (width 0) (type default) (color 0 0 0 0))
+  )
+  (wire (pts (xy 63.5 129.54) (xy 63.5 119.38))
+    (stroke (width 0) (type default) (color 0 0 0 0))
+  )
   (wire (pts (xy 25.4 66.04) (xy 73.66 66.04))
     (stroke (width 0) (type default) (color 0 0 0 0))
   )
-  (wire (pts (xy 25.4 66.04) (xy 25.4 116.84))
-    (stroke (width 0) (type default) (color 0 0 0 0))
-  )
-  (wire (pts (xy 55.88 53.34) (xy 73.66 53.34))
-    (stroke (width 0) (type default) (color 0 0 0 0))
-  )
-  (wire (pts (xy 60.96 109.22) (xy 60.96 78.74))
-    (stroke (width 0) (type default) (color 0 0 0 0))
-  )
-  (wire (pts (xy 63.5 96.52) (xy 63.5 111.76))
-    (stroke (width 0) (type default) (color 0 0 0 0))
-  )
-  (wire (pts (xy 63.5 129.54) (xy 71.12 129.54))
-    (stroke (width 0) (type default) (color 0 0 0 0))
-  )
-  (wire (pts (xy 71.12 134.62) (xy 71.12 129.54))
-    (stroke (width 0) (type default) (color 0 0 0 0))
-  )
-  (wire (pts (xy 68.58 152.4) (xy 71.12 152.4))
-    (stroke (width 0) (type default) (color 0 0 0 0))
-  )
-  (wire (pts (xy 91.44 86.36) (xy 111.76 86.36))
-    (stroke (width 0) (type default) (color 0 0 0 0))
-  )
-  (wire (pts (xy 58.42 68.58) (xy 58.42 86.36))
-    (stroke (width 0) (type default) (color 0 0 0 0))
-  )
-  (wire (pts (xy 78.74 48.26) (xy 55.88 48.26))
-    (stroke (width 0) (type default) (color 0 0 0 0))
-  )
-  (wire (pts (xy 66.04 111.76) (xy 63.5 111.76))
-    (stroke (width 0) (type default) (color 0 0 0 0))
-  )
-  (wire (pts (xy 78.74 50.8) (xy 55.88 50.8))
-    (stroke (width 0) (type default) (color 0 0 0 0))
-  )
-  (wire (pts (xy 63.5 129.54) (xy 63.5 119.38))
-    (stroke (width 0) (type default) (color 0 0 0 0))
-  )
   (wire (pts (xy 78.74 35.56) (xy 55.88 35.56))
     (stroke (width 0) (type default) (color 0 0 0 0))
@@
     (stroke (width 0) (type default) (color 0 0 0 0))
   )
+  (wire (pts (xy 73.66 66.04) (xy 120.65 66.04))
+    (stroke (width 0) (type default) (color 0 0 0 0))
+  )
   (wire (pts (xy 78.74 45.72) (xy 55.88 45.72))
     (stroke (width 0) (type default) (color 0 0 0 0))
@@
     (effects (font (size 1.27 1.27)) (justify left bottom))
   )
-  (text "Temporarily, K8 (dst_wr_en)\nis directly connected to U101 pin 10.\nThis allows the microcodeto enable\nregister writes when YARC has control."
+  (text "Temporarily, K8 (dst_wr_en)\nis directly connected to U101 pin 10.\nThis allows the microcodeto enable\nregister writes when NANO# has control."
     (at 20.32 129.54 0)
     (effects (font (size 1.27 1.27)) (justify left bottom))
@@
     (effects (font (size 1.27 1.27)) (justify left bottom))
   )
+  (text "A second 7-pin physical connector\nis located adjacent to the 6-pin\nthat brings signals from the Nano."
+    (at 15.24 62.23 0)
+    (effects (font (size 1.27 1.27)) (justify left bottom))
+  )
   (text "This sheet summarizes the use of the YARC kludge space,\nwhich is located north of the main system memory. Some\nlogic from the kludge space appears on other sheets."
     (at 167.64 182.88 0)
@@
     )
   )
+  (global_label "YARC{slash}~{NANO} to ALU Control" (shape input) (at 120.65 66.04 0) (fields_autoplaced)
+    (effects (font (size 1.27 1.27)) (justify left))
+    (property "Intersheet References" "${INTERSHEET_REFS}" (id 0) (at 149.3098 65.9606 0)
+      (effects (font (size 1.27 1.27)) (justify left) hide)
+    )
+  )

Commit message: Ongoing corrections. Document the Nano's sysbus enable control for the first time.
Connections:
- net GND: no longer U101.5 (I0b)
- net ~{BUS_EN}: now reaches U101.7 (Zb)
- new net MCR bit 0x04 (bit 2): U101.5 (I0b)
Changed lines of the file:
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@@
   (junction (at 78.74 78.74) (diameter 0) (color 0 0 0 0)
   )
-  (junction (at 63.5 96.52) (diameter 0) (color 0 0 0 0)
-  )
   (junction (at 63.5 111.76) (diameter 0) (color 0 0 0 0)
   )
@@
     (stroke (width 0) (type default) (color 0 0 0 0))
   )
-  (wire (pts (xy 66.04 93.98) (xy 63.5 93.98))
-    (stroke (width 0) (type default) (color 0 0 0 0))
-  )
   (wire (pts (xy 58.42 86.36) (xy 66.04 86.36))
     (stroke (width 0) (type default) (color 0 0 0 0))
@@
     (stroke (width 0) (type default) (color 0 0 0 0))
   )
-  (wire (pts (xy 91.44 109.22) (xy 129.54 109.22))
+  (wire (pts (xy 91.44 109.22) (xy 132.08 109.22))
     (stroke (width 0) (type default) (color 0 0 0 0))
   )
@@
     (stroke (width 0) (type default) (color 0 0 0 0))
   )
+  (wire (pts (xy 53.34 93.98) (xy 66.04 93.98))
+    (stroke (width 0) (type default) (color 0 0 0 0))
+  )
   (wire (pts (xy 58.42 68.58) (xy 58.42 86.36))
     (stroke (width 0) (type default) (color 0 0 0 0))
@@
     (stroke (width 0) (type default) (color 0 0 0 0))
   )
+  (wire (pts (xy 91.44 93.98) (xy 132.08 93.98))
+    (stroke (width 0) (type default) (color 0 0 0 0))
+  )
   (wire (pts (xy 66.04 88.9) (xy 53.34 88.9))
     (stroke (width 0) (type default) (color 0 0 0 0))
@@
     (stroke (width 0) (type default) (color 0 0 0 0))
   )
-  (wire (pts (xy 63.5 93.98) (xy 63.5 96.52))
-    (stroke (width 0) (type default) (color 0 0 0 0))
-  )
   (wire (pts (xy 66.04 104.14) (xy 53.34 104.14))
     (stroke (width 0) (type default) (color 0 0 0 0))
@@
     (stroke (width 0) (type default) (color 0 0 0 0))
   )
-  (wire (pts (xy 127 83.82) (xy 139.7 83.82))
-    (stroke (width 0) (type default) (color 0 0 0 0))
-  )
-  (wire (pts (xy 66.04 96.52) (xy 63.5 96.52))
+  (wire (pts (xy 127 83.82) (xy 132.08 83.82))
     (stroke (width 0) (type default) (color 0 0 0 0))
   )
@@
     (stroke (width 0) (type default) (color 0 0 0 0))
   )
-  (wire (pts (xy 91.44 101.6) (xy 127 101.6))
+  (wire (pts (xy 91.44 101.6) (xy 132.08 101.6))
     (stroke (width 0) (type default) (color 0 0 0 0))
   )
   (wire (pts (xy 78.74 129.54) (xy 78.74 127))
+    (stroke (width 0) (type default) (color 0 0 0 0))
+  )
+  (wire (pts (xy 63.5 96.52) (xy 66.04 96.52))
     (stroke (width 0) (type default) (color 0 0 0 0))
   )
@@
     )
   )
+  (global_label "MCR bit 0x04 (bit 2)" (shape input) (at 53.34 93.98 180) (fields_autoplaced)
+    (effects (font (size 1.27 1.27)) (justify right))
+    (property "Intersheet References" "${INTERSHEET_REFS}" (id 0) (at 30.5464 93.9006 0)
+      (effects (font (size 1.27 1.27)) (justify right) hide)
+    )
+  )
   (global_label "MCR bit 0x80 (bit 7)" (shape input) (at 53.34 101.6 180) (fields_autoplaced)
     (effects (font (size 1.27 1.27)) (justify right))
@@
     )
   )
-  (global_label "~{DST_EN} to U96B" (shape input) (at 127 101.6 0) (fields_autoplaced)
-    (effects (font (size 1.27 1.27)) (justify left))
-    (property "Intersheet References" "${INTERSHEET_REFS}" (id 0) (at 145.1369 101.5206 0)
+  (global_label "~{DST_EN} to U96B" (shape input) (at 132.08 101.6 0) (fields_autoplaced)
+    (effects (font (size 1.27 1.27)) (justify left))
+    (property "Intersheet References" "${INTERSHEET_REFS}" (id 0) (at 150.2169 101.5206 0)
       (effects (font (size 1.27 1.27)) (justify left) hide)
     )
@@
     )
   )
-  (global_label "~{ADDRESS_XCVR_EN}" (shape input) (at 129.54 109.22 0) (fields_autoplaced)
-    (effects (font (size 1.27 1.27)) (justify left))
-    (property "Intersheet References" "${INTERSHEET_REFS}" (id 0) (at 149.6726 109.1406 0)
+  (global_label "~{ADDRESS_XCVR_EN}" (shape input) (at 132.08 109.22 0) (fields_autoplaced)
+    (effects (font (size 1.27 1.27)) (justify left))
+    (property "Intersheet References" "${INTERSHEET_REFS}" (id 0) (at 152.2126 109.1406 0)
       (effects (font (size 1.27 1.27)) (justify left) hide)
     )
@@
     )
   )
+  (global_label "~{BUS_EN}" (shape input) (at 132.08 93.98 0) (fields_autoplaced)
+    (effects (font (size 1.27 1.27)) (justify left))
+    (property "Intersheet References" "${INTERSHEET_REFS}" (id 0) (at 141.7502 93.9006 0)
+      (effects (font (size 1.27 1.27)) (justify left) hide)
+    )
+  )
   (global_label "SYSCLK" (shape input) (at 104.14 81.28 180) (fields_autoplaced)
     (effects (font (size 1.27 1.27)) (justify right))
@@
     )
   )
-  (global_label "IR_CLK" (shape input) (at 139.7 83.82 0) (fields_autoplaced)
-    (effects (font (size 1.27 1.27)) (justify left))
-    (property "Intersheet References" "${INTERSHEET_REFS}" (id 0) (at 148.5236 83.7406 0)
-      (effects (font (size 1.27 1.27)) (justify left) hide)
-    )
+  (global_label "IR_CLK" (shape input) (at 132.08 83.82 0) (fields_autoplaced)
+    (effects (font (size 1.27 1.27)) (justify left))
+    (property "Intersheet References" "${INTERSHEET_REFS}" (id 0) (at 140.9036 83.7406 0)
+      (effects (font (size 1.27 1.27)) (justify left) hide)
+    )

Commit message: Continuing corrections (only - no new functionality)
Connections:
- net ACR_CLK NANO DECODER 0x02 (bit 1): no longer J8.2 (Pin_2)
- new net NOT USED: J8.2 (Pin_2)
Changed lines of the file:
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@@
     (stroke (width 0) (type default) (color 0 0 0 0))
   )
-  (wire (pts (xy 111.76 43.18) (xy 55.88 43.18))
+  (wire (pts (xy 119.38 43.18) (xy 55.88 43.18))
     (stroke (width 0) (type default) (color 0 0 0 0))
   )
@@
     (stroke (width 0) (type default) (color 0 0 0 0))
   )
-  (wire (pts (xy 111.76 68.58) (xy 111.76 43.18))
+  (wire (pts (xy 119.38 68.58) (xy 119.38 43.18))
     (stroke (width 0) (type default) (color 0 0 0 0))
   )
@@
     (stroke (width 0) (type default) (color 0 0 0 0))
   )
-  (wire (pts (xy 73.66 66.04) (xy 120.65 66.04))
+  (wire (pts (xy 73.66 66.04) (xy 78.74 66.04))
     (stroke (width 0) (type default) (color 0 0 0 0))
   )
@@
     (stroke (width 0) (type default) (color 0 0 0 0))
   )
-  (wire (pts (xy 58.42 68.58) (xy 111.76 68.58))
+  (wire (pts (xy 58.42 68.58) (xy 119.38 68.58))
     (stroke (width 0) (type default) (color 0 0 0 0))
   )
@@
     )
   )
-  (global_label "YARC{slash}~{NANO} to ALU Control" (shape input) (at 120.65 66.04 0) (fields_autoplaced)
-    (effects (font (size 1.27 1.27)) (justify left))
-    (property "Intersheet References" "${INTERSHEET_REFS}" (id 0) (at 149.3098 65.9606 0)
+  (global_label "YARC{slash}~{NANO} to ALU Control" (shape input) (at 78.74 66.04 0) (fields_autoplaced)
+    (effects (font (size 1.27 1.27)) (justify left))
+    (property "Intersheet References" "${INTERSHEET_REFS}" (id 0) (at 107.3998 65.9606 0)
       (effects (font (size 1.27 1.27)) (justify left) hide)
     )
@@
     )
   )
-  (global_label "NOT USED" (shape input) (at 78.74 48.26 0) (fields_autoplaced)
-    (effects (font (size 1.27 1.27)) (justify left))
-    (property "Intersheet References" "${INTERSHEET_REFS}" (id 0) (at 90.7083 48.1806 0)
-      (effects (font (size 1.27 1.27)) (justify left) hide)
-    )
+  (global_label "ACR_CLK sheet 14 (North Central)" (shape input) (at 78.74 48.26 0) (fields_autoplaced)
+    (effects (font (size 1.27 1.27)) (justify left))
+    (property "Intersheet References" "${INTERSHEET_REFS}" (id 0) (at 114.3545 48.1806 0)
+      (effects (font (size 1.27 1.27)) (justify left) hide)
+    )
