File: ki/YARC/ALU.kicad_sch (KiCad schematic)
At the start: 7 parts, among them U116 AS6C6264, U117 AS6C6264, U118 AS6C6264, U119 74LS245, U120 74LS245, U121 74LS573, U122 74LS574

Commit message: Ongoing corrections and improvements. No major additions.
Changed lines of the file:
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@@
       (effects (font (size 1.27 1.27)) hide)
     )
-    (property "Value" "GND" (id 1) (at 231.14 114.3 0))
+    (property "Value" "GND" (id 1) (at 241.3 114.3 0))
     (property "Footprint" "" (id 2) (at 236.22 114.3 0)
       (effects (font (size 1.27 1.27)) hide)
