File: ki/YARC/NorthCentral.kicad_sch (KiCad schematic)
At the start: 10 parts, among them U102 74HC245, U103 74HC245, U106 74LS139, U128 74LS157, U132 74LS157, U133 74LS21, U134 74LS32, U138 74LS14

Commit message: Removed about 2/3 of 2300+ errors from the ERC
Changed lines of the file:
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@@
+    (stroke (width 0) (type default))
+  )
+  (bus (pts (xy 15.24 144.78) (xy 15.24 153.67))
     (stroke (width 0) (type default))
   )
@@
     (stroke (width 0) (type default))
   )
-  (bus (pts (xy 12.7 20.32) (xy 22.86 20.32))
+  (bus (pts (xy 15.24 20.32) (xy 22.86 20.32))
     (stroke (width 0) (type default))
   )
@@
     (stroke (width 0) (type default))
   )
-  (bus (pts (xy 12.7 144.78) (xy 22.86 144.78))
+  (bus (pts (xy 15.24 144.78) (xy 22.86 144.78))
     (stroke (width 0) (type default))
   )
   (wire (pts (xy 132.08 33.02) (xy 132.08 63.5))
+    (stroke (width 0) (type default))
+  )
+  (bus (pts (xy 15.24 20.32) (xy 15.24 30.48))
     (stroke (width 0) (type default))
   )
@@
     (effects (font (size 1.27 1.27)) (justify left bottom))
   )
-  (label "SYSADDR14" (at 66.04 43.18 0)
-    (effects (font (size 1.27 1.27)) (justify left bottom))
-  )
-  (label "SYSADDR1" (at 66.04 83.82 0)
-    (effects (font (size 1.27 1.27)) (justify left bottom))
-  )
-  (label "S1BUS2" (at 31.75 86.36 0)
+  (label "SYSADDR14" (at 66.04 43.18 0) (fields_autoplaced)
+    (effects (font (size 1.27 1.27)) (justify left bottom))
+  )
+  (label "SYSADDR1" (at 66.04 83.82 0) (fields_autoplaced)
+    (effects (font (size 1.27 1.27)) (justify left bottom))
+  )
+  (label "S1BUS2" (at 31.75 86.36 0) (fields_autoplaced)
     (effects (font (size 1.27 1.27)) (justify left bottom))
   )
@@
     (effects (font (size 1.27 1.27)) (justify left bottom))
   )
-  (label "KX4" (at 36.83 167.64 0)
-    (effects (font (size 1.27 1.27)) (justify left bottom))
-  )
-  (label "S1BUS12" (at 31.75 38.1 0)
+  (label "KX4" (at 36.83 167.64 0) (fields_autoplaced)
+    (effects (font (size 1.27 1.27)) (justify left bottom))
+  )
+  (label "S1BUS12" (at 31.75 38.1 0) (fields_autoplaced)
     (effects (font (size 1.27 1.27)) (justify left bottom))
   )
@@
     (effects (font (size 1.27 1.27)) (justify left bottom))
   )
-  (label "S1BUS5" (at 31.75 93.98 0)
+  (label "S1BUS5" (at 31.75 93.98 0) (fields_autoplaced)
     (effects (font (size 1.27 1.27)) (justify left bottom))
   )
@@
     (effects (font (size 1.27 1.27)) (justify left bottom))
   )
-  (label "S1BUS10" (at 31.75 33.02 0)
-    (effects (font (size 1.27 1.27)) (justify left bottom))
-  )
-  (label "S1BUS[0..15]" (at 12.7 20.32 0) (fields_autoplaced)
-    (effects (font (size 1.27 1.27)) (justify left bottom))
-  )
-  (label "KX3" (at 36.83 165.1 0)
-    (effects (font (size 1.27 1.27)) (justify left bottom))
-  )
-  (label "KX2" (at 36.83 162.56 0)
-    (effects (font (size 1.27 1.27)) (justify left bottom))
-  )
-  (label "KX6" (at 36.83 172.72 0)
-    (effects (font (size 1.27 1.27)) (justify left bottom))
-  )
-  (label "S1BUS9" (at 31.75 30.48 0)
-    (effects (font (size 1.27 1.27)) (justify left bottom))
-  )
-  (label "SYSADDR11" (at 66.04 35.56 0)
-    (effects (font (size 1.27 1.27)) (justify left bottom))
-  )
-  (label "KX5" (at 36.83 170.18 0)
-    (effects (font (size 1.27 1.27)) (justify left bottom))
-  )
-  (label "S1BUS6" (at 31.75 96.52 0)
+  (label "S1BUS10" (at 31.75 33.02 0) (fields_autoplaced)
+    (effects (font (size 1.27 1.27)) (justify left bottom))
+  )
+  (label "KX3" (at 36.83 165.1 0) (fields_autoplaced)
+    (effects (font (size 1.27 1.27)) (justify left bottom))
+  )
+  (label "KX2" (at 36.83 162.56 0) (fields_autoplaced)
+    (effects (font (size 1.27 1.27)) (justify left bottom))
+  )
+  (label "KX6" (at 36.83 172.72 0) (fields_autoplaced)
+    (effects (font (size 1.27 1.27)) (justify left bottom))
+  )
+  (label "S1BUS9" (at 31.75 30.48 0) (fields_autoplaced)
+    (effects (font (size 1.27 1.27)) (justify left bottom))
+  )
+  (label "SYSADDR11" (at 66.04 35.56 0) (fields_autoplaced)
+    (effects (font (size 1.27 1.27)) (justify left bottom))
+  )
+  (label "KX5" (at 36.83 170.18 0) (fields_autoplaced)
+    (effects (font (size 1.27 1.27)) (justify left bottom))
+  )
+  (label "S1BUS6" (at 31.75 96.52 0) (fields_autoplaced)
     (effects (font (size 1.27 1.27)) (justify left bottom))
   )
@@
     (effects (font (size 1.27 1.27)) (justify left bottom))
   )
-  (label "KX1" (at 36.83 160.02 0)
-    (effects (font (size 1.27 1.27)) (justify left bottom))
-  )
-  (label "S1BUS1" (at 31.75 83.82 0)
+  (label "KX1" (at 36.83 160.02 0) (fields_autoplaced)
+    (effects (font (size 1.27 1.27)) (justify left bottom))
+  )
+  (label "S1BUS1" (at 31.75 83.82 0) (fields_autoplaced)
     (effects (font (size 1.27 1.27)) (justify left bottom))
   )
@@
     (effects (font (size 1.27 1.27)) (justify right bottom))
   )
-  (label "SYSADDR12" (at 66.04 38.1 0)
-    (effects (font (size 1.27 1.27)) (justify left bottom))
-  )
-  (label "SYSADDR3" (at 66.04 88.9 0)
-    (effects (font (size 1.27 1.27)) (justify left bottom))
-  )
-  (label "SYSADDR2" (at 66.04 86.36 0)
-    (effects (font (size 1.27 1.27)) (justify left bottom))
-  )
-  (label "S1BUS4" (at 31.75 91.44 0)
+  (label "SYSADDR12" (at 66.04 38.1 0) (fields_autoplaced)
+    (effects (font (size 1.27 1.27)) (justify left bottom))
+  )
+  (label "SYSADDR3" (at 66.04 88.9 0) (fields_autoplaced)
+    (effects (font (size 1.27 1.27)) (justify left bottom))
+  )
+  (label "SYSADDR2" (at 66.04 86.36 0) (fields_autoplaced)
+    (effects (font (size 1.27 1.27)) (justify left bottom))
+  )
+  (label "S1BUS4" (at 31.75 91.44 0) (fields_autoplaced)
     (effects (font (size 1.27 1.27)) (justify left bottom))
   )
@@
     (effects (font (size 1.27 1.27)) (justify right bottom))
   )
-  (label "S1BUS3" (at 31.75 88.9 0)
-    (effects (font (size 1.27 1.27)) (justify left bottom))
-  )
-  (label "SYSADDR4" (at 66.04 91.44 0)
+  (label "S1BUS3" (at 31.75 88.9 0) (fields_autoplaced)
+    (effects (font (size 1.27 1.27)) (justify left bottom))
+  )
+  (label "SYSADDR4" (at 66.04 91.44 0) (fields_autoplaced)
     (effects (font (size 1.27 1.27)) (justify left bottom))
   )
@@
     (effects (font (size 1.27 1.27)) (justify right bottom))
   )
-  (label "SYSADDR10" (at 66.04 33.02 0)
+  (label "SYSADDR10" (at 66.04 33.02 0) (fields_autoplaced)
     (effects (font (size 1.27 1.27)) (justify left bottom))
   )
@@
     (effects (font (size 1.27 1.27)) (justify right bottom))
   )
-  (label "SYSADDR13" (at 66.04 40.64 0)
-    (effects (font (size 1.27 1.27)) (justify left bottom))
-  )
-  (label "SYSADDR[0..15]" (at 78.74 20.32 0) (fields_autoplaced)
+  (label "SYSADDR13" (at 66.04 40.64 0) (fields_autoplaced)
     (effects (font (size 1.27 1.27)) (justify left bottom))
   )
@@
     (effects (font (size 1.27 1.27)) (justify right bottom))
   )
-  (label "KX[0..7]" (at 12.7 144.78 0) (fields_autoplaced)
-    (effects (font (size 1.27 1.27)) (justify left bottom))
-  )
   (label "SYSADDR0" (at 66.04 81.28 0) (fields_autoplaced)
     (effects (font (size 1.27 1.27)) (justify left bottom))
@@
     (effects (font (size 1.27 1.27)) (justify left bottom))
   )
-  (label "S1BUS14" (at 31.75 43.18 0)
+  (label "S1BUS14" (at 31.75 43.18 0) (fields_autoplaced)
     (effects (font (size 1.27 1.27)) (justify left bottom))
   )
@@
     (effects (font (size 1.27 1.27)) (justify left bottom))
   )
-  (label "SYSADDR9" (at 66.04 30.48 0)
-    (effects (font (size 1.27 1.27)) (justify left bottom))
-  )
-  (label "SYSADDR6" (at 66.04 96.52 0)
-    (effects (font (size 1.27 1.27)) (justify left bottom))
-  )
-  (label "S1BUS11" (at 31.75 35.56 0)
-    (effects (font (size 1.27 1.27)) (justify left bottom))
-  )
-  (label "S1BUS13" (at 31.75 40.64 0)
+  (label "SYSADDR9" (at 66.04 30.48 0) (fields_autoplaced)
+    (effects (font (size 1.27 1.27)) (justify left bottom))
+  )
+  (label "SYSADDR6" (at 66.04 96.52 0) (fields_autoplaced)
+    (effects (font (size 1.27 1.27)) (justify left bottom))
+  )
+  (label "S1BUS11" (at 31.75 35.56 0) (fields_autoplaced)
+    (effects (font (size 1.27 1.27)) (justify left bottom))
+  )
+  (label "S1BUS13" (at 31.75 40.64 0) (fields_autoplaced)
     (effects (font (size 1.27 1.27)) (justify left bottom))
   )
@@
     (effects (font (size 1.27 1.27)) (justify right bottom))
   )
-  (label "SYSADDR5" (at 66.04 93.98 0)
+  (label "SYSADDR5" (at 66.04 93.98 0) (fields_autoplaced)
     (effects (font (size 1.27 1.27)) (justify left bottom))
   )
@@
     )
   )
+  (global_label "SYSADDR[0..15]" (shape input) (at 83.82 20.32 0) (fields_autoplaced)
+    (effects (font (size 1.27 1.27)) (justify left))
+    (property "Intersheetrefs" "${INTERSHEET_REFS}" (at 101.7429 20.32 0)
+      (effects (font (size 1.27 1.27)) (justify left) hide)
+    )
+  )
   (global_label "~{RAM_C1_OE}" (shape input) (at 203.2 45.72 0) (fields_autoplaced)
     (effects (font (size 1.27 1.27)) (justify left))
@@
     )
   )
+  (global_label "S1BUS[0..15]" (shape input) (at 15.24 30.48 270) (fields_autoplaced)
+    (effects (font (size 1.27 1.27)) (justify right))
+    (property "Intersheetrefs" "${INTERSHEET_REFS}" (at 15.24 46.2257 90)
+      (effects (font (size 1.27 1.27)) (justify right) hide)
+    )
+  )
   (global_label "SYSCLK" (shape input) (at 153.67 81.28 180) (fields_autoplaced)
     (effects (font (size 1.27 1.27)) (justify right))
@@
       (effects (font (size 1.27 1.27)) (justify right) hide)
     )
+  )
+  (global_label "KX[0..7]" (shape input) (at 15.24 153.67 270) (fields_autoplaced)
+    (effects (font (size 1.27 1.27)) (justify right))
+    (property "Intersheetrefs" "${INTERSHEET_REFS}" (at 15.24 164.4567 90)
+      (effects (font (size 1.27 1.27)) (justify right) hide)
+    )

Commit message: Ongoing fixes for ERC errors
Parts:
- gave numbers to parts that had none: 2
Changed lines of the file:
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@@
   (symbol (lib_id "74xx:74LS32") (at 256.54 152.4 0) (unit 5)
     (in_bom yes) (on_board yes) (dnp no)
-    (property "Reference" "U?" (at 248.92 142.24 0)
+    (property "Reference" "U147" (at 248.92 142.24 0)
       (effects (font (size 1.27 1.27)) (justify left))
     )
@@
       (project "YARC"
         (path "/22e0f8e1-b0d7-4d47-bb7c-8ef04cd95fca/51c42971-ddd1-444d-b989-88f84ae04d0f"
-          (reference "U?") (unit 5)
+          (reference "U147") (unit 5)
         )
       )
@@
   (symbol (lib_id "74xx:74LS574") (at 53.34 170.18 0) (unit 1)
     (in_bom yes) (on_board yes) (dnp no) (fields_autoplaced)
-    (property "Reference" "U?" (at 55.3594 149.86 0)
+    (property "Reference" "U146" (at 55.3594 149.86 0)
       (effects (font (size 1.27 1.27)) (justify left))
     )
@@
       (project "YARC"
         (path "/22e0f8e1-b0d7-4d47-bb7c-8ef04cd95fca/51c42971-ddd1-444d-b989-88f84ae04d0f"
-          (reference "U?") (unit 1)
-        )
-      )
+          (reference "U146") (unit 1)
+        )
+      )

Commit message: Ongoing schematic changes
Parts:
- removed U147: 74LS32, symbol 74xx:74LS32
- added U93: 74LS32, symbol 74xx:74LS32
Connections:
- net GND: now also U93.7 (GND)
- net VCC: now also U93.14 (VCC)
- net ~{ADDRESS_XCVR_EN} renamed ~{GRtoA}
- no-connect marks 0 -> 2
Other:
- note removed: "This control is essentially YARC/NANO#. When YARC has control, it is always low."
Changed lines of the file:
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@@
   (junction (at 246.38 128.27) (diameter 0) (color 0 0 0 0)
   )
+  (junction (at 256.54 165.1) (diameter 0) (color 0 0 0 0)
+  )
   (junction (at 167.64 139.7) (diameter 0) (color 0 0 0 0)
   )
   (junction (at 129.54 106.68) (diameter 0) (color 0 0 0 0)
   )
-  (junction (at 256.54 165.1) (diameter 0) (color 0 0 0 0)
-  )
   (junction (at 152.4 114.3) (diameter 0) (color 0 0 0 0)
   )
@@
   (junction (at 27.94 50.8) (diameter 0) (color 0 0 0 0)
   )
+  (junction (at 256.54 139.7) (diameter 0) (color 0 0 0 0)
+  )
   (junction (at 30.48 106.68) (diameter 0) (color 0 0 0 0)
   )
-  (junction (at 256.54 139.7) (diameter 0) (color 0 0 0 0)
-  )
   (junction (at 104.14 99.06) (diameter 0) (color 0 0 0 0)
   )
@@
   (junction (at 185.42 81.28) (diameter 0) (color 0 0 0 0)
   )
+  (no_connect (at 261.62 128.27))
+  (no_connect (at 261.62 114.3))
   (bus_entry (at 78.74 86.36) (size -2.54 -2.54)
     (stroke (width 0) (type default))
@@
     (at 81.28 175.26 0)
     (effects (font (size 1.524 1.524)) (justify left bottom))
-  )
-  (text "This control is essentially\nYARC/NANO#. When YARC has\ncontrol, it is always low."
-    (at 34.29 132.08 0)
-    (effects (font (size 1.27 1.27)) (justify left bottom))
   )
   (text "ALU CONTROL REGISTER (ACR)" (at 38.1 200.66 0)
@@
     )
   )
-  (global_label "~{ADDRESS_XCVR_EN}" (shape input) (at 30.48 111.76 270) (fields_autoplaced)
+  (global_label "~{GRtoA}" (shape input) (at 30.48 111.76 270) (fields_autoplaced)
     (effects (font (size 1.27 1.27)) (justify right))
-    (property "Intersheetrefs" "${INTERSHEET_REFS}" (at 30.5594 131.8926 90)
+    (property "Intersheetrefs" "${INTERSHEET_REFS}" (at 30.48 120.2485 90)
       (effects (font (size 1.27 1.27)) (justify right) hide)
     )
@@
         (path "/22e0f8e1-b0d7-4d47-bb7c-8ef04cd95fca/51c42971-ddd1-444d-b989-88f84ae04d0f"
           (reference "U138") (unit 7)
-        )
-      )
-    )
-  )
-  (symbol (lib_id "74xx:74LS32") (at 256.54 152.4 0) (unit 5)
-    (in_bom yes) (on_board yes) (dnp no)
-    (property "Reference" "U147" (at 248.92 142.24 0)
-      (effects (font (size 1.27 1.27)) (justify left))
-    )
-    (property "Value" "74LS32" (at 254 152.4 0)
-      (effects (font (size 1.27 1.27)) (justify left))
-    )
-    (property "Footprint" "" (at 256.54 152.4 0)
-      (effects (font (size 1.27 1.27)) hide)
-    )
-    (property "Datasheet" "http://www.ti.com/lit/gpn/sn74LS32" (at 256.54 152.4 0)
-      (effects (font (size 1.27 1.27)) hide)
-    )
-    (pin "1")
-    (pin "2")
-    (pin "3")
-    (pin "4")
-    (pin "5")
-    (pin "6")
-    (pin "10")
-    (pin "8")
-    (pin "9")
-    (pin "11")
-    (pin "12")
-    (pin "13")
-    (pin "14")
-    (pin "7")
-    (instances
-      (project "YARC"
-        (path "/22e0f8e1-b0d7-4d47-bb7c-8ef04cd95fca/51c42971-ddd1-444d-b989-88f84ae04d0f"
-          (reference "U147") (unit 5)
         )
       )
@@
     )
   )
-  (symbol (lib_id "74xx:74LS32") (at 195.58 88.9 0) (mirror x) (unit 2)
+  (symbol (lib_id "74xx:74LS32") (at 256.54 152.4 0) (unit 5)
     (in_bom yes) (on_board yes) (dnp no)
-    (property "Reference" "U134" (at 200.66 85.09 0)
-      (effects (font (size 1.27 1.27)))
-    )
-    (property "Value" "74LS32" (at 195.58 88.9 0)
-      (effects (font (size 1.27 1.27)))
-    )
-    (property "Footprint" "" (at 195.58 88.9 0)
-      (effects (font (size 1.27 1.27)) hide)
-    )
-    (property "Datasheet" "http://www.ti.com/lit/gpn/sn74LS32" (at 195.58 88.9 0)
+    (property "Reference" "U93" (at 257.81 143.51 0)
+      (effects (font (size 1.27 1.27)) (justify left))
+    )
+    (property "Value" "74LS32" (at 252.73 152.4 0)
+      (effects (font (size 1.27 1.27)) (justify left))
+    )
+    (property "Footprint" "" (at 256.54 152.4 0)
+      (effects (font (size 1.27 1.27)) hide)
+    )
+    (property "Datasheet" "http://www.ti.com/lit/gpn/sn74LS32" (at 256.54 152.4 0)
       (effects (font (size 1.27 1.27)) hide)
     )
@@
     (instances
       (project "YARC"
+        (path "/22e0f8e1-b0d7-4d47-bb7c-8ef04cd95fca/abd64d43-20ca-4b37-94fd-5fc041c76dd4"
+          (reference "U93") (unit 5)
+        )
+        (path "/22e0f8e1-b0d7-4d47-bb7c-8ef04cd95fca/51c42971-ddd1-444d-b989-88f84ae04d0f"
+          (reference "U147") (unit 5)
+        )
+      )
+    )
+  )
+  (symbol (lib_id "74xx:74LS32") (at 195.58 88.9 0) (mirror x) (unit 2)
+    (in_bom yes) (on_board yes) (dnp no)
+    (property "Reference" "U134" (at 200.66 85.09 0)
+      (effects (font (size 1.27 1.27)))
+    )
+    (property "Value" "74LS32" (at 195.58 88.9 0)
+      (effects (font (size 1.27 1.27)))
+    )
+    (property "Footprint" "" (at 195.58 88.9 0)
+      (effects (font (size 1.27 1.27)) hide)
+    )
+    (property "Datasheet" "http://www.ti.com/lit/gpn/sn74LS32" (at 195.58 88.9 0)
+      (effects (font (size 1.27 1.27)) hide)
+    )
+    (pin "1")
+    (pin "2")
+    (pin "3")
+    (pin "4")
+    (pin "5")
+    (pin "6")
+    (pin "10")
+    (pin "8")
+    (pin "9")
+    (pin "11")
+    (pin "12")
+    (pin "13")
+    (pin "14")
+    (pin "7")
+    (instances
+      (project "YARC"
         (path "/22e0f8e1-b0d7-4d47-bb7c-8ef04cd95fca/51c42971-ddd1-444d-b989-88f84ae04d0f"
           (reference "U134") (unit 2)
@@
   )
   (symbol (lib_id "74xx:74LS21") (at 241.3 152.4 0) (unit 3)
-    (in_bom yes) (on_board yes) (dnp no) (fields_autoplaced)
-    (property "Reference" "U133" (at 247.65 151.1299 0)
+    (in_bom yes) (on_board yes) (dnp no)
+    (property "Reference" "U133" (at 242.57 143.51 0)
       (effects (font (size 1.27 1.27)) (justify left))
     )
-    (property "Value" "74LS21" (at 247.65 153.6699 0)
+    (property "Value" "74LS21" (at 238.76 152.4 0)
       (effects (font (size 1.27 1.27)) (justify left))
     )
