File: ki/YARC/SouthCentral.kicad_sch (KiCad schematic)
At the start: 9 parts, among them U104 74LS86, U83 74LS139, U84 74LS157, U85 74LS157, U86 74LS157, U87 74LS138, U88 74HC00, U89 74LS157, U90 74LS157

Commit message: Disable sysaddr_src decoder when the Nano has control of the address bus (the Nano never disables its address transceivers when it has control)
Parts:
- removed unit 2 of U104
Connections:
- no-connect marks 9 -> 8
Changed lines of the file:
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@@
   (junction (at 210.82 132.08) (diameter 0) (color 0 0 0 0)
   )
-  (junction (at 182.88 177.8) (diameter 0) (color 0 0 0 0)
-  )
   (junction (at 210.82 55.88) (diameter 0) (color 0 0 0 0)
   )
@@
   )
   (junction (at 226.06 83.82) (diameter 0) (color 0 0 0 0)
-  )
-  (junction (at 182.88 167.64) (diameter 0) (color 0 0 0 0)
   )
   (junction (at 180.34 157.48) (diameter 0) (color 0 0 0 0)
@@
   (no_connect (at 154.94 147.32))
   (no_connect (at 154.94 144.78))
-  (no_connect (at 198.12 180.34))
   (no_connect (at 154.94 149.86))
   (bus_entry (at 127 157.48) (size -2.54 2.54)
@@
     (stroke (width 0) (type default))
   )
-  (wire (pts (xy 165.1 167.64) (xy 182.88 167.64))
+  (wire (pts (xy 165.1 167.64) (xy 210.82 167.64))
     (stroke (width 0) (type default))
   )
@@
     (stroke (width 0) (type default))
   )
-  (wire (pts (xy 182.88 182.88) (xy 182.88 177.8))
-    (stroke (width 0) (type default))
-  )
   (wire (pts (xy 129.54 149.86) (xy 129.54 157.48))
     (stroke (width 0) (type default))
@@
     (stroke (width 0) (type default))
   )
-  (wire (pts (xy 182.88 177.8) (xy 182.88 167.64))
-    (stroke (width 0) (type default))
-  )
   (wire (pts (xy 213.36 40.64) (xy 210.82 40.64))
     (stroke (width 0) (type default))
@@
   )
   (wire (pts (xy 60.96 147.32) (xy 60.96 175.26))
-    (stroke (width 0) (type default))
-  )
-  (wire (pts (xy 182.88 167.64) (xy 210.82 167.64))
     (stroke (width 0) (type default))
   )
@@
         )
       )
-    )
-  )
-  (symbol (lib_id "74xx:74LS86") (at 190.5 180.34 0) (unit 2)
-    (in_bom yes) (on_board yes) (dnp no)
-    (property "Reference" "U104" (at 195.58 175.26 0)
-      (effects (font (size 1.27 1.27)))
-    )
-    (property "Value" "74LS86" (at 190.5 180.34 0)
-      (effects (font (size 1.27 1.27)))
-    )
-    (property "Footprint" "" (at 190.5 180.34 0)
-      (effects (font (size 1.27 1.27)) hide)
-    )
-    (property "Datasheet" "74xx/74ls86.pdf" (at 190.5 180.34 0)
-      (effects (font (size 1.27 1.27)) hide)
-    )
-    (pin "1")
-    (pin "2")
-    (pin "3")
-    (pin "4")
-    (pin "5")
-    (pin "6")
-    (pin "10")
-    (pin "8")
-    (pin "9")
-    (pin "11")
-    (pin "12")
-    (pin "13")
-    (pin "14")
-    (pin "7")
-    (instances
-      (project "YARC"
-        (path "/22e0f8e1-b0d7-4d47-bb7c-8ef04cd95fca/89d830c1-f0d9-4d89-9863-428a1b54ae3d"
-          (reference "U104") (unit 2)
-        )
-      )
