File: pcb/V501/V501.kicad_pcb (KiCad board)
At the start: 4 copper layers, 25.7 x 76.6 mm, 10 parts, among them J1 Conn_01x30_Pin, J2 Conn_01x30_Pin, U1 74LS670, U2 74LS670, U3 74LS670, U4 74LS670

Commit message: Minor updates and polish for V501.
Routing:
- net VCC: track 139.6 -> 147.2 mm
- net GND: track 106.3 -> 110.1 mm
Other:
- board size 25.7 x 76.6 mm -> 25.4 x 76.6 mm
