File: pcb/V501/V501.kicad_sch (KiCad schematic)
At the start: 10 parts, among them J1 Conn_01x30_Pin, J2 Conn_01x30_Pin, U1 74LS670, U2 74LS670, U3 74LS670, U4 74LS670

Commit message: Minor updates and polish for V501.
Other:
- title: V501 -> V501 Quad 16-bit D latch (address registers)
