File: pcb/V503/LowerHalf.kicad_sch (KiCad schematic)
At the start: 9 parts, among them J1 Conn_01x20_Pin, J2 Conn_01x20_Pin, J3 Conn_01x20_Pin, J4 Conn_01x20_Pin, J5 Conn_01x30_Pin, U11 74LS245, U12 74LS245, U13 74LS245, U14 74LS245

Commit message: Clean up clearances, run DRC and ERC, and generate Gerbers. Tape out.
Parts:
- removed J5: Conn_01x30_Pin, Connector_PinHeader_2.54mm:PinHeader_1x30_P2.54mm_Vertical, symbol Connector:Conn_01x30_Pin
Changed lines of the file:
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@@
-    )
-  )
-  (symbol (lib_id "Connector:Conn_01x30_Pin") (at 193.04 102.87 0) (unit 1)
-    (in_bom yes) (on_board yes) (dnp no) (fields_autoplaced)
-    (property "Reference" "J5" (at 193.675 62.23 0)
-      (effects (font (size 1.27 1.27)))
-    )
-    (property "Value" "Conn_01x30_Pin" (at 193.675 64.77 0)
-      (effects (font (size 1.27 1.27)))
-    )
-    (property "Footprint" "Connector_PinHeader_2.54mm:PinHeader_1x30_P2.54mm_Vertical" (at 193.04 102.87 0)
-      (effects (font (size 1.27 1.27)) hide)
-    )
-    (property "Datasheet" "~" (at 193.04 102.87 0)
-      (effects (font (size 1.27 1.27)) hide)
-    )
-    (pin "1")
-    (pin "10")
-    (pin "11")
-    (pin "12")
-    (pin "13")
-    (pin "14")
-    (pin "15")
-    (pin "16")
-    (pin "17")
-    (pin "18")
-    (pin "19")
-    (pin "2")
-    (pin "20")
-    (pin "21")
-    (pin "22")
-    (pin "23")
-    (pin "24")
-    (pin "25")
-    (pin "26")
-    (pin "27")
-    (pin "28")
-    (pin "29")
-    (pin "3")
-    (pin "30")
-    (pin "4")
-    (pin "5")
-    (pin "6")
-    (pin "7")
-    (pin "8")
-    (pin "9")
-    (instances
-      (project "V503"
-        (path "/d60807f5-1f73-4a51-8f52-ff2764d64fa5/9b1d77fd-a71f-49f6-9744-75ce4d8ca94f"
-          (reference "J5") (unit 1)
-        )
-      )
     )
   )
